Commit message: wip acea

File: concert_isaac/python/src/concert_isaac/assets/urdf/concert_complete.urdf (robot description, URDF)
Before this commit: robot ModularBot, 78 links, 77 joints
Links:
- link J1_A_stator: geometry collision mesh filename=file:///workspace/concert_isaac/assets/meshes/concert/simpl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 scale=0.001 0.001 0.001; visual mesh filename=file:///workspace/concert_isaac/assets/meshes/concert/conce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 scale=0.001 0.001 0.001
- link J1_B_stator: geometry collision mesh filename=file:///workspace/concert_isaac/assets/meshes/concert/simpl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 scale=0.001 0.001 0.001; visual mesh filename=file:///workspace/concert_isaac/assets/meshes/concert/conce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 scale=0.001 0.001 0.001
- link J1_C_stator: geometry collision mesh filename=file:///workspace/concert_isaac/assets/meshes/concert/simpl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 scale=0.001 0.001 0.001; visual mesh filename=file:///workspace/concert_isaac/assets/meshes/concert/conce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 scale=0.001 0.001 0.001
- link J1_D_stator: geometry collision mesh filename=file:///workspace/concert_isaac/assets/meshes/concert/simpl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 scale=0.001 0.001 0.001; visual mesh filename=file:///workspace/concert_isaac/assets/meshes/concert/conce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 scale=0.001 0.001 0.001
- link J1_E_stator: geometry collision mesh filename=file:///workspace/concert_isaac/assets/meshes/concert/simpl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 scale=0.001 0.001 0.001; visual mesh filename=file:///workspace/concert_isaac/assets/meshes/concert/conce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 scale=0.001 0.001 0.001
- link J2_E_stator: geometry collision mesh filename=file:///workspace/concert_isaac/assets/meshes/concert/simpl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 scale=0.001 0.001 0.001; visual mesh filename=file:///workspace/concert_isaac/assets/meshes/concert/conce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 scale=0.001 0.001 0.001
- link J3_E_stator: geometry collision mesh filename=file:///workspace/concert_isaac/assets/meshes/concert/simpl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 scale=0.001 0.001 0.001; visual mesh filename=file:///workspace/concert_isaac/assets/meshes/concert/conce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 scale=0.001 0.001 0.001
- link J4_E_stator: geometry collision mesh filename=file:///workspace/concert_isaac/assets/meshes/concert/simpl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 scale=0.001 0.001 0.001; visual mesh filename=file:///workspace/concert_isaac/assets/meshes/concert/conce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 scale=0.001 0.001 0.001
- link J5_E_stator: geometry collision mesh filename=file:///workspace/concert_isaac/assets/meshes/concert/simpl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 scale=0.001 0.001 0.001; visual mesh filename=file:///workspace/concert_isaac/assets/meshes/concert/conce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 scale=0.001 0.001 0.001
- link J6_E_stator: geometry collision mesh filename=file:///workspace/concert_isaac/assets/meshes/concert/simpl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 scale=0.001 0.001 0.001; visual mesh filename=file:///workspace/concert_isaac/assets/meshes/concert/conce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 scale=0.001 0.001 0.001
- link L_1_A: geometry collision mesh filename=file:///workspace/concert_isaac/assets/meshes/concert/simpl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 scale=0.001 0.001 0.001; visual mesh filename=file:///workspace/concert_isaac/assets/meshes/concert/conce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 scale=0.001 0.001 0.001
- link L_1_B: geometry collision mesh filename=file:///workspace/concert_isaac/assets/meshes/concert/simpl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 scale=0.001 0.001 0.001; visual mesh filename=file:///workspace/concert_isaac/assets/meshes/concert/conce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 scale=0.001 0.001 0.001
- link L_1_C: geometry collision mesh filename=file:///workspace/concert_isaac/assets/meshes/concert/simpl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 scale=0.001 0.001 0.001; visual mesh filename=file:///workspace/concert_isaac/assets/meshes/concert/conce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 scale=0.001 0.001 0.001
- link L_1_D: geometry collision mesh filename=file:///workspace/concert_isaac/assets/meshes/concert/simpl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 scale=0.001 0.001 0.001; visual mesh filename=file:///workspace/concert_isaac/assets/meshes/concert/conce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 scale=0.001 0.001 0.001
- link L_1_E: geometry collision mesh filename=file:///workspace/concert_isaac/assets/meshes/concert/simpl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 scale=0.001 0.001 0.001; visual mesh filename=file:///workspace/concert_isaac/assets/meshes/concert/conce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 scale=0.001 0.001 0.001
- link L_2_E: geometry collision mesh filename=file:///workspace/concert_isaac/assets/meshes/concert/simpl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 scale=0.001 0.001 0.001; visual mesh filename=file:///workspace/concert_isaac/assets/meshes/concert/conce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 scale=0.001 0.001 0.001
- link L_3_E: geometry collision mesh filename=file:///workspace/concert_isaac/assets/meshes/concert/simpl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 scale=0.001 0.001 0.001; visual mesh filename=file:///workspace/concert_isaac/assets/meshes/concert/conce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 scale=0.001 0.001 0.001
- link L_3_link_1_E: geometry collision cylinder length=0.4 radius=0.0675; visual mesh filename=file:///workspace/concert_isaac/assets/meshes/concert/mesh_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 scale=0.001 0.001 0.001
- link L_4_E: geometry collision mesh filename=file:///workspace/concert_isaac/assets/meshes/concert/simpl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 scale=0.001 0.001 0.001; visual mesh filename=file:///workspace/concert_isaac/assets/meshes/concert/conce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 scale=0.001 0.001 0.001
- link L_5_E: geometry collision mesh filename=file:///workspace/concert_isaac/assets/meshes/concert/simpl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 scale=0.001 0.001 0.001; visual mesh filename=file:///workspace/concert_isaac/assets/meshes/concert/conce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 scale=0.001 0.001 0.001
- link L_5_link_1_E: geometry collision cylinder length=0.4 radius=0.0675; visual mesh filename=file:///workspace/concert_isaac/assets/meshes/concert/mesh_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 scale=0.001 0.001 0.001
- link L_6_E: geometry collision mesh filename=file:///workspace/concert_isaac/assets/meshes/concert/simpl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 scale=0.001 0.001 0.001; visual mesh filename=file:///workspace/concert_isaac/assets/meshes/concert/conce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 scale=0.001 0.001 0.001
- link end_effector_E: geometry collision mesh filename=file:///workspace/concert_isaac/assets/meshes/concert/simpl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 scale=0.001 0.001 0.001; visual mesh filename=file:///workspace/concert_isaac/assets/meshes/concert/passi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 scale=0.001 0.001 0.001
- link mobile_base: geometry collision mesh filename=file:///workspace/concert_isaac/assets/meshes/concert/simpl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 scale=0.001 0.001 0.001; visual mesh filename=file:///workspace/concert_isaac/assets/meshes/concert/conce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 scale=0.001 0.001 0.001
- link wheel_A: geometry collision cylinder length=0.1 radius=0.16; visual mesh filename=file:///workspace/concert_isaac/assets/meshes/concert/conce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 scale=0.001 0.001 0.001
- link wheel_B: geometry collision cylinder length=0.1 radius=0.16; visual mesh filename=file:///workspace/concert_isaac/assets/meshes/concert/conce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 scale=0.001 0.001 0.001
- link wheel_C: geometry collision cylinder length=0.1 radius=0.16; visual mesh filename=file:///workspace/concert_isaac/assets/meshes/concert/conce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 scale=0.001 0.001 0.001
- link wheel_D: geometry collision cylinder length=0.1 radius=0.16; visual mesh filename=file:///workspace/concert_isaac/assets/meshes/concert/conce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 scale=0.001 0.001 0.001
